File: Checkpoint1/Esquematico/esquematico.kicad_sch (KiCad schematic)
At the start: 29 parts, among them Q1 BC547, Q10 BC547, Q2 BC547, Q3 BC547, Q4 BC547, Q5 BC557, Q6 BC557, Q7 TIP42C, Q8 BC337, Q9 BC547, U1 LM358, U2 TL431D

Commit message: Refactor code structure for improved readability and maintainability
Parts:
- added unit 3 of U1
- R1, R2: value R -> 100
- R4, R5, RVRS+: value R -> 10k
- R6: value R -> 100k
- R7: value R -> 1k
- RF1, RF2: value R -> 470k
- RL: value R -> 4
- RS: value R -> 0.1
- RVO+, RVO-: value R -> 454k
- RVREF, RVREF+: value R -> 625k
- RVRS-: renamed from RRVRS-; value R -> 10k
- Rref: renamed from R3; value R -> 1k2
- U1: footprint Package_DFN_QFN:DFN-8-1EP_2x2mm_P0.5mm_EP1.05x1.75mm -> (none)
- renumbered U2 to VREF
Connections:
- net GND: now also Q4.3 (E), R4.1, RL.2, RVO+.2, RVREF+.2, U1.4 (V-); no longer Q4.1 (C)
- net Vb: now reaches Q2.1 (C), Q8.2 (B)
- net Vb: now also Q10.1 (C), Q6.1 (C); no longer Q6.3 (E)
- net VREG: now reaches R1.1, R2.1
- net VREG: now also Q1.2 (B), Q7.3 (E), Rref.1, VREF.1 (K), VREF.8 (REF), U1.8 (V+); no longer Q7.2 (C)
- net VRS: now reaches Q8.3 (E), RS.1
- net VRS: now also Q7.2 (C), RVRS+.2; no longer Q7.3 (E)
- net Vo: now reaches R5.1, RL.1, RS.2
- net Vo: now also RVO-.2, RVRS-.2
- net VREF: now reaches RVREF.2
- net VREF: now also R6.2
- net at R2.2: now also Q6.3 (E); no longer Q6.1 (C)
- net at Q3.2 (B), Q4.2 (B), Rref.2: now also Q4.1 (C); no longer Q4.3 (E)
Other:
- moved on the sheet: Q4, Rref

Commit message: Update subproject commit and modify schematic value
Parts:
- RL: value 4 -> 50
Changed lines of the file:
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@@
 			)
 		)
-		(property "Value" "4"
+		(property "Value" "50"
 			(at 159.258 93.98 0)
 			(show_name no)
