File: Checkpoint1/Esquematico/esquematico.kicad_pcb (KiCad board)
At the start: 2 copper layers, 115 x 60 mm, 38 parts, among them J1 Conn_01x02, J2 Conn_01x02, Q1 BC547, Q10 BC547, Q2 BC547, Q3 BC547, Q4 BC547, Q5 BC557, Q6 BC557, Q7 TIP42C, Q8 BC337, Q9 BC547, U1 LM358, U2 TL431LP

Commit message: Nuevo PCB
Parts:
- moved Q7 6.80 mm to (145.5, 58.0), turned to 180 degrees
Routing:
- net VRS: track 50.3 -> 59.1 mm
- net Net-(Q7-B): track 11.4 -> 17.9 mm
- net Net-(R7-Pad1): track 41.1 -> 39.0 mm
- net VREG: track 64.6 -> 65.1 mm
