File: Checkpoint2/Esquematico/esquematico.kicad_pcb (KiCad board)
At the start: 2 copper layers, 115 x 60 mm, 38 parts, among them J1 Conn_01x02, J2 Conn_01x02, Q1 BC547, Q10 BC547, Q2 BC547, Q3 BC547, Q4 BC547, Q5 BC557, Q6 BC557, Q7 TIP42C, Q8 BC337, Q9 BC547, U1 LM358, U2 TL431LP

Commit message: Nuevo PCB
Parts:
- RS1: footprint Resistor_THT:R_Axial_DIN0309_L9.0mm_D3.2mm_P12.70mm_Horizontal -> Resistor_THT:R_Axial_Power_L25.0mm_W6.4mm_P27.94mm
- moved RS1 46.2 mm to (213.0, 109.0), turned to 90 degrees
- moved R6 10.2 mm to (202.5, 89.2), turned to -90 degrees
- moved RF2 8.43 mm to (195.3, 87.5)
- moved Q9 7.83 mm to (186.5, 96.8)
- moved RVO+1 7.66 mm to (182.7, 81.0)
- moved Q7 6.56 mm to (139.9, 59.0), turned to 0 degrees
- moved R5 5.61 mm to (178.8, 88.5)
- moved RVREF1 4.00 mm to (200.8, 57.0)
- moved RVREF+1 3.01 mm to (200.9, 77.0)
- moved RVO-1 2.50 mm to (213.7, 64.0)
- moved RVRS-1 2.01 mm to (213.7, 70.5)
- moved J2 1.53 mm to (176.0, 103.0)
- moved R7 1.51 mm to (182.8, 64.0)
- moved RF1 1.51 mm to (182.8, 57.0)
- moved RVRS+1 1.51 mm to (195.5, 70.0)
Routing:
- net Net-(JP4-A): track 26.4 -> 104.3 mm
- net VREF: track 237.6 -> 259.4 mm
- net Vo: track 92.5 -> 74.1 mm
- net Net-(Q9-B): track 28.3 -> 20.9 mm
- net Net-(Q7-B): track 11.4 -> 18.4 mm
- net Net-(U1A--): track 76.8 -> 72.5 mm
- net Net-(R7-Pad1): track 41.1 -> 37.2 mm
- net VREG: track 64.6 -> 68.3 mm
- net Net-(Q10-B): track 34.8 -> 31.3 mm
- net Net-(JP3-B): track 17.8 -> 16.1 mm
- net VRS: track 50.3 -> 51.9 mm
- net Net-(JP3-A): track 23.7 -> 24.3 mm
- net Net-(U1A-+): track 81.0 -> 81.6 mm
