File: Checkpoint2/Esquematico/esquematico.kicad_sch (KiCad schematic)
At the start: 38 parts, among them J1 Conn_01x02, J2 Conn_01x02, Q1 BC547, Q10 BC547, Q2 BC547, Q3 BC547, Q4 BC547, Q5 BC557, Q6 BC557, Q7 TIP42C, Q8 BC337, Q9 BC547, U1 LM358, U2 TL431LP

Commit message: Nuevo PCB
Parts:
- RS1: footprint Resistor_THT:R_Axial_DIN0309_L9.0mm_D3.2mm_P12.70mm_Horizontal -> Resistor_THT:R_Axial_Power_L25.0mm_W6.4mm_P27.94mm
Changed lines of the file:
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@@
 			)
 		)
-		(property "Footprint" "Resistor_THT:R_Axial_DIN0309_L9.0mm_D3.2mm_P12.70mm_Horizontal"
+		(property "Footprint" "Resistor_THT:R_Axial_Power_L25.0mm_W6.4mm_P27.94mm"
 			(at 155.702 83.82 90)
 			(hide yes)
